Commit message: included contact force reward

File: quadrup.urdf (robot description, URDF)
Before this commit: robot bipedal, 13 links, 12 joints
Joints:
- joint bl_bicep_to_thigh: limit lower=-0.785 upper=0.785 effort=20 velocity=2 -> lower=-0.785 upper=0.785 effort=11 velocity=2
- joint bl_shoulder_to_base: limit lower=-0.785 upper=0.785 effort=20 velocity=2 -> lower=-0.785 upper=0.785 effort=11 velocity=2
- joint bl_thigh_to_shoulder: limit lower=-0.785 upper=0.785 effort=20 velocity=2 -> lower=-0.785 upper=0.785 effort=11 velocity=2
- joint br_bicep_to_thigh: limit lower=-0.785 upper=0.785 effort=20 velocity=2 -> lower=-0.785 upper=0.785 effort=11 velocity=2
- joint br_shoulder_to_base: limit lower=-0.785 upper=0.785 effort=20 velocity=2 -> lower=-0.785 upper=0.785 effort=11 velocity=2
- joint br_thigh_to_shoulder: limit lower=-0.785 upper=0.785 effort=20 velocity=2 -> lower=-0.785 upper=0.785 effort=11 velocity=2
- joint fl_bicep_to_thigh: limit lower=-0.785 upper=0.785 effort=20 velocity=2 -> lower=-0.785 upper=0.785 effort=11 velocity=2
- joint fl_shoulder_to_base: limit lower=-0.785 upper=0.785 effort=20 velocity=2 -> lower=-0.785 upper=0.785 effort=11 velocity=2
- joint fl_thigh_to_shoulder: limit lower=-0.785 upper=0.785 effort=20 velocity=2 -> lower=-0.785 upper=0.785 effort=11 velocity=2
- joint fr_bicep_to_thigh: limit lower=-0.785 upper=0.785 effort=20 velocity=2 -> lower=-0.785 upper=0.785 effort=11 velocity=2
- joint fr_shoulder_to_base: limit lower=-0.785 upper=0.785 effort=20 velocity=2 -> lower=-0.785 upper=0.785 effort=11 velocity=2
- joint fr_thigh_to_shoulder: limit lower=-0.785 upper=0.785 effort=20 velocity=2 -> lower=-0.785 upper=0.785 effort=11 velocity=2

Commit message: change floor color

File: quadrup.urdf (robot description, URDF)
Before this commit: robot bipedal, 13 links, 12 joints
Links:
- link base_link: mass 1. -> 2.
- link bl_bicep: mass 0.1 -> 1
- link bl_shoulder: mass 0.1 -> 1
- link bl_thigh: mass 0.1 -> 1
- link br_bicep: mass 0.1 -> 1
- link br_shoulder: mass 0.1 -> 1
- link br_thigh: mass 0.1 -> 1
- link fl_bicep: mass 0.1 -> 1
- link fl_shoulder: mass 0.1 -> 1
- link fl_thigh: mass 0.1 -> 1
- link fr_bicep: mass 0.1 -> 1
- link fr_shoulder: mass 0.1 -> 1
- link fr_thigh: mass 0.1 -> 1

Commit message: increase torque for each leg and in crease swing angle of  each leg and T value

File: quadrup.urdf (robot description, URDF)
Before this commit: robot bipedal, 13 links, 12 joints
Joints:
- joint bl_bicep_to_thigh: limit lower=-0.785 upper=0.785 effort=11 velocity=2 -> lower=-0.785 upper=0.785 effort=15 velocity=2
- joint bl_shoulder_to_base: limit lower=-0.785 upper=0.785 effort=11 velocity=2 -> lower=-0.785 upper=0.785 effort=15 velocity=2
- joint bl_thigh_to_shoulder: limit lower=-0.785 upper=0.785 effort=11 velocity=2 -> lower=-0.785 upper=0.785 effort=15 velocity=2
- joint br_bicep_to_thigh: limit lower=-0.785 upper=0.785 effort=11 velocity=2 -> lower=-0.785 upper=0.785 effort=15 velocity=2
- joint br_shoulder_to_base: limit lower=-0.785 upper=0.785 effort=11 velocity=2 -> lower=-0.785 upper=0.785 effort=15 velocity=2
- joint br_thigh_to_shoulder: limit lower=-0.785 upper=0.785 effort=11 velocity=2 -> lower=-0.785 upper=0.785 effort=15 velocity=2
- joint fl_bicep_to_thigh: limit lower=-0.785 upper=0.785 effort=11 velocity=2 -> lower=-0.785 upper=0.785 effort=15 velocity=2
- joint fl_shoulder_to_base: limit lower=-0.785 upper=0.785 effort=11 velocity=2 -> lower=-0.785 upper=0.785 effort=15 velocity=2
- joint fl_thigh_to_shoulder: limit lower=-0.785 upper=0.785 effort=11 velocity=2 -> lower=-0.785 upper=0.785 effort=15 velocity=2
- joint fr_bicep_to_thigh: limit lower=-0.785 upper=0.785 effort=11 velocity=2 -> lower=-0.785 upper=0.785 effort=15 velocity=2
- joint fr_shoulder_to_base: limit lower=-0.785 upper=0.785 effort=11 velocity=2 -> lower=-0.785 upper=0.785 effort=15 velocity=2
- joint fr_thigh_to_shoulder: limit lower=-0.785 upper=0.785 effort=11 velocity=2 -> lower=-0.785 upper=0.785 effort=15 velocity=2

Commit message: increase torque for each leg and in crease swing angle of  each leg and T value

File: quadrup.urdf (robot description, URDF)
Before this commit: robot bipedal, 13 links, 12 joints
Joints:
- joint bl_bicep_to_thigh: limit lower=-0.785 upper=0.785 effort=15 velocity=2 -> lower=-0.785 upper=0.785 effort=11 velocity=2
- joint bl_shoulder_to_base: limit lower=-0.785 upper=0.785 effort=15 velocity=2 -> lower=-0.785 upper=0.785 effort=11 velocity=2
- joint bl_thigh_to_shoulder: limit lower=-0.785 upper=0.785 effort=15 velocity=2 -> lower=-0.785 upper=0.785 effort=11 velocity=2
- joint br_bicep_to_thigh: limit lower=-0.785 upper=0.785 effort=15 velocity=2 -> lower=-0.785 upper=0.785 effort=11 velocity=2
- joint br_shoulder_to_base: limit lower=-0.785 upper=0.785 effort=15 velocity=2 -> lower=-0.785 upper=0.785 effort=11 velocity=2
- joint br_thigh_to_shoulder: limit lower=-0.785 upper=0.785 effort=15 velocity=2 -> lower=-0.785 upper=0.785 effort=11 velocity=2
- joint fl_bicep_to_thigh: limit lower=-0.785 upper=0.785 effort=15 velocity=2 -> lower=-0.785 upper=0.785 effort=11 velocity=2
- joint fl_shoulder_to_base: limit lower=-0.785 upper=0.785 effort=15 velocity=2 -> lower=-0.785 upper=0.785 effort=11 velocity=2
- joint fl_thigh_to_shoulder: limit lower=-0.785 upper=0.785 effort=15 velocity=2 -> lower=-0.785 upper=0.785 effort=11 velocity=2
- joint fr_bicep_to_thigh: limit lower=-0.785 upper=0.785 effort=15 velocity=2 -> lower=-0.785 upper=0.785 effort=11 velocity=2
- joint fr_shoulder_to_base: limit lower=-0.785 upper=0.785 effort=15 velocity=2 -> lower=-0.785 upper=0.785 effort=11 velocity=2
- joint fr_thigh_to_shoulder: limit lower=-0.785 upper=0.785 effort=15 velocity=2 -> lower=-0.785 upper=0.785 effort=11 velocity=2

Commit message: add more engine power

File: quadrup.urdf (robot description, URDF)
Before this commit: robot bipedal, 13 links, 12 joints
Joints:
- joint bl_bicep_to_thigh: limit lower=-0.785 upper=0.785 effort=11 velocity=2 -> lower=-0.785 upper=0.785 effort=20 velocity=2
- joint bl_shoulder_to_base: limit lower=-0.785 upper=0.785 effort=11 velocity=2 -> lower=-0.785 upper=0.785 effort=20 velocity=2
- joint bl_thigh_to_shoulder: limit lower=-0.785 upper=0.785 effort=11 velocity=2 -> lower=-0.785 upper=0.785 effort=20 velocity=2
- joint br_bicep_to_thigh: limit lower=-0.785 upper=0.785 effort=11 velocity=2 -> lower=-0.785 upper=0.785 effort=20 velocity=2
- joint br_shoulder_to_base: limit lower=-0.785 upper=0.785 effort=11 velocity=2 -> lower=-0.785 upper=0.785 effort=20 velocity=2
- joint br_thigh_to_shoulder: limit lower=-0.785 upper=0.785 effort=11 velocity=2 -> lower=-0.785 upper=0.785 effort=20 velocity=2
- joint fl_bicep_to_thigh: limit lower=-0.785 upper=0.785 effort=11 velocity=2 -> lower=-0.785 upper=0.785 effort=20 velocity=2
- joint fl_shoulder_to_base: limit lower=-0.785 upper=0.785 effort=11 velocity=2 -> lower=-0.785 upper=0.785 effort=20 velocity=2
- joint fl_thigh_to_shoulder: limit lower=-0.785 upper=0.785 effort=11 velocity=2 -> lower=-0.785 upper=0.785 effort=20 velocity=2
- joint fr_bicep_to_thigh: limit lower=-0.785 upper=0.785 effort=11 velocity=2 -> lower=-0.785 upper=0.785 effort=20 velocity=2
- joint fr_shoulder_to_base: limit lower=-0.785 upper=0.785 effort=11 velocity=2 -> lower=-0.785 upper=0.785 effort=20 velocity=2
- joint fr_thigh_to_shoulder: limit lower=-0.785 upper=0.785 effort=11 velocity=2 -> lower=-0.785 upper=0.785 effort=20 velocity=2

Commit message: add more engine power

File: quadrup.urdf (robot description, URDF)
Before this commit: robot bipedal, 13 links, 12 joints
Joints:
- joint bl_bicep_to_thigh: limit lower=-0.785 upper=0.785 effort=20 velocity=2 -> lower=-0.785 upper=0.785 effort=15 velocity=2
- joint bl_shoulder_to_base: limit lower=-0.785 upper=0.785 effort=20 velocity=2 -> lower=-0.785 upper=0.785 effort=15 velocity=2
- joint bl_thigh_to_shoulder: limit lower=-0.785 upper=0.785 effort=20 velocity=2 -> lower=-0.785 upper=0.785 effort=15 velocity=2
- joint br_bicep_to_thigh: limit lower=-0.785 upper=0.785 effort=20 velocity=2 -> lower=-0.785 upper=0.785 effort=15 velocity=2
- joint br_shoulder_to_base: limit lower=-0.785 upper=0.785 effort=20 velocity=2 -> lower=-0.785 upper=0.785 effort=15 velocity=2
- joint br_thigh_to_shoulder: limit lower=-0.785 upper=0.785 effort=20 velocity=2 -> lower=-0.785 upper=0.785 effort=15 velocity=2
- joint fl_bicep_to_thigh: limit lower=-0.785 upper=0.785 effort=20 velocity=2 -> lower=-0.785 upper=0.785 effort=15 velocity=2
- joint fl_shoulder_to_base: limit lower=-0.785 upper=0.785 effort=20 velocity=2 -> lower=-0.785 upper=0.785 effort=15 velocity=2
- joint fl_thigh_to_shoulder: limit lower=-0.785 upper=0.785 effort=20 velocity=2 -> lower=-0.785 upper=0.785 effort=15 velocity=2
- joint fr_bicep_to_thigh: limit lower=-0.785 upper=0.785 effort=20 velocity=2 -> lower=-0.785 upper=0.785 effort=15 velocity=2
- joint fr_shoulder_to_base: limit lower=-0.785 upper=0.785 effort=20 velocity=2 -> lower=-0.785 upper=0.785 effort=15 velocity=2
- joint fr_thigh_to_shoulder: limit lower=-0.785 upper=0.785 effort=20 velocity=2 -> lower=-0.785 upper=0.785 effort=15 velocity=2
