Commit message: Add files via upload

File: quadrupv1.urdf (robot description, URDF)
Before this commit: robot bipedal, 13 links, 12 joints
Links:
- link base_link: mass 1. -> 1.5
- link bl_bicep: geometry collision box size=0.03 0.03 0.115; collision sphere radius=0.03
- link bl_thigh: geometry collision box size=0.05 0.05 0.08; visual box size=0.05 0.05 0.08
- link br_bicep: geometry collision box size=0.03 0.03 0.115; collision sphere radius=0.03
- link br_thigh: geometry collision box size=0.05 0.05 0.08; visual box size=0.05 0.05 0.08
- link fl_bicep: geometry collision box size=0.03 0.03 0.115; collision sphere radius=0.03
- link fl_thigh: geometry collision box size=0.05 0.05 0.08; visual box size=0.05 0.05 0.08
- link fr_bicep: geometry collision box size=0.03 0.03 0.115; collision sphere radius=0.03
- link fr_thigh: geometry collision box size=0.05 0.05 0.08; visual box size=0.05 0.05 0.08
Joints:
- joint bl_bicep_to_thigh: limit lower=-0.785 upper=0.785 effort=11 velocity=2 -> lower=-0.785 upper=0.785 effort=0.9 velocity=2
- joint bl_shoulder_to_base: limit lower=-0.785 upper=0.785 effort=11 velocity=2 -> lower=-0.785 upper=0.785 effort=0.9 velocity=2
- joint bl_thigh_to_shoulder: limit lower=-0.785 upper=0.785 effort=11 velocity=2 -> lower=-0.785 upper=0.785 effort=0.9 velocity=2
- joint br_bicep_to_thigh: limit lower=-0.785 upper=0.785 effort=11 velocity=2 -> lower=-0.785 upper=0.785 effort=0.9 velocity=2
- joint br_shoulder_to_base: limit lower=-0.785 upper=0.785 effort=11 velocity=2 -> lower=-0.785 upper=0.785 effort=0.9 velocity=2
- joint br_thigh_to_shoulder: limit lower=-0.785 upper=0.785 effort=11 velocity=2 -> lower=-0.785 upper=0.785 effort=0.9 velocity=2
- joint fl_bicep_to_thigh: limit lower=-0.785 upper=0.785 effort=11 velocity=2 -> lower=-0.785 upper=0.785 effort=0.9 velocity=2
- joint fl_shoulder_to_base: limit lower=-0.785 upper=0.785 effort=11 velocity=2 -> lower=-0.785 upper=0.785 effort=0.9 velocity=2
- joint fl_thigh_to_shoulder: limit lower=-0.785 upper=0.785 effort=11 velocity=2 -> lower=-0.785 upper=0.785 effort=0.9 velocity=2
- joint fr_bicep_to_thigh: limit lower=-0.785 upper=0.785 effort=11 velocity=2 -> lower=-0.785 upper=0.785 effort=0.9 velocity=2
- joint fr_shoulder_to_base: limit lower=-0.785 upper=0.785 effort=11 velocity=2 -> lower=-0.785 upper=0.785 effort=0.9 velocity=2
- joint fr_thigh_to_shoulder: limit lower=-0.785 upper=0.785 effort=11 velocity=2 -> lower=-0.785 upper=0.785 effort=0.9 velocity=2
