Commit message: Update NCKH_AN_and_NHAN.urdf

File: NCKH_AN_and_NHAN/urdf/NCKH_AN_and_NHAN.urdf (robot description, URDF)
Before this commit: robot NCKH_AN_and_NHAN, 13 links, 12 joints
Joints:
- joint wl1.joint1: limit lower=-1.571 upper=1.571 effort=0.9 velocity=2 -> lower=-1.571 upper=1.571 effort=2 velocity=2
- joint wl1.joint2: limit lower=-1.571 upper=1.571 effort=0.9 velocity=2 -> lower=-1.571 upper=1.571 effort=2 velocity=2
- joint wl1.joint3: limit lower=-1.571 upper=1.571 effort=0.9 velocity=2 -> lower=-1.571 upper=1.571 effort=2 velocity=2
- joint wl2.joint1: limit lower=-1.571 upper=1.571 effort=0.9 velocity=2 -> lower=-1.571 upper=1.571 effort=2 velocity=2
- joint wl2.joint2: limit lower=-1.571 upper=1.571 effort=0.9 velocity=2 -> lower=-1.571 upper=1.571 effort=2 velocity=2
- joint wl2.joint3: limit lower=-1.571 upper=1.571 effort=0.9 velocity=2 -> lower=-1.571 upper=1.571 effort=2 velocity=2
- joint wl3.joint1: limit lower=-1.571 upper=1.571 effort=0.9 velocity=2 -> lower=-1.571 upper=1.571 effort=2 velocity=2
- joint wl3.joint2: limit lower=-1.571 upper=1.571 effort=0.9 velocity=2 -> lower=-1.571 upper=1.571 effort=2 velocity=2
- joint wl3.joint3: limit lower=-1.571 upper=1.571 effort=0.9 velocity=2 -> lower=-1.571 upper=1.571 effort=2 velocity=2
- joint wl4.joint1: limit lower=-1.571 upper=1.571 effort=0.9 velocity=2 -> lower=-1.571 upper=1.571 effort=2 velocity=2
- joint wl4.joint2: limit lower=-1.571 upper=1.571 effort=0.9 velocity=2 -> lower=-1.571 upper=1.571 effort=2 velocity=2
- joint wl4.joint3: limit lower=-1.571 upper=1.571 effort=0.9 velocity=2 -> lower=-1.571 upper=1.571 effort=2 velocity=2
